File: 445pcb_round3.kicad_sch (KiCad schematic)
At the start: 40 parts, among them J1 LED, J2 LED, J3 LED, J4 SG3, J5 SG4, J6 SG5, J7 SG6, U1 ICM-20948, U2 LM358_DFN, U3 ATmega328P-A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

Commit message: Add files via upload
Parts:
- added J11: SG1, Connector_Molex:Molex_KK-254_AE-6410-02A_1x02_P2.54mm_Vertical, symbol Connector_Generic:Conn_01x02
- added J13: LED, Connector_Molex:Molex_KK-254_AE-6410-02A_1x02_P2.54mm_Vertical, symbol Connector_Generic:Conn_01x02
- added P1: USB_C_Plug_USB2.0, Connector_USB:USB_C_Plug_Molex_105444, symbol Connector:USB_C_Plug_USB2.0
- added R25: 1k, Resistor_SMD:R_0805_2012Metric_Pad1.20x1.40mm_HandSolder, symbol Device:R
- added SW1: SW_SPST, Button_Switch_THT:SW_DIP_SPSTx01_Slide_9.78x4.72mm_W7.62mm_P2.54mm, symbol Switch:SW_SPST
- C2: footprint (none) -> Capacitor_SMD:C_0805_2012Metric_Pad1.18x1.45mm_HandSolder
- R8: footprint (none) -> Resistor_SMD:R_0805_2012Metric_Pad1.20x1.40mm_HandSolder
- gave numbers to parts that had none: 11
Connections:
- net +5V: now also J13.1 (Pin_1), R25.2
- net GND: now also J13.2 (Pin_2), P1.A1 (GND), P1.A12 (GND), P1.B1 (GND), P1.B12 (GND)
- net at R3.1: now also U3.1 (PD3); no longer U3.30 (PD0)
- net UART TXD: now reaches U3.31 (PD1)
- net UART TXD: now also P1.A6 (D+)
- new net: P1.A4 (VBUS), P1.A9 (VBUS), P1.B4 (VBUS), P1.B9 (VBUS)
- new net: J11.2 (Pin_2), R25.1, SW1.2 (B)
- new net: J11.1 (Pin_1), SW1.1 (A)
- new net UART RXD: P1.A7 (D-), U3.30 (PD0)
Other:
- moved on the sheet: C2, J10, J2, J3, R10, R11, R12, R13, R14, R15, R16, R19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

Commit message: adding power to op-amps, switching USB to connector, zener diode
Parts:
- removed P1: USB_C_Plug_USB2.0, Connector_USB:USB_C_Plug_Molex_105444, symbol Connector:USB_C_Plug_USB2.0
- removed R11, R12, R22, R23: 3.3M, Resistor_SMD:R_0805_2012Metric_Pad1.20x1.40mm_HandSolder, symbol Device:R
- removed R20, R21, R9: 10k, Resistor_SMD:R_0805_2012Metric_Pad1.20x1.40mm_HandSolder, symbol Device:R
- removed U2, U4, U5: LM358_DFN, Package_DFN_QFN:DFN-8-1EP_2x2mm_P0.5mm_EP1.05x1.75mm, symbol Amplifier_Operational:LM358_DFN
- added D2: MBR0520, Diode_SMD:D_SOD-123, symbol Diode:MBR0520
- added J19: Conn_01x04_Pin, Connector_Molex:Molex_KK-254_AE-6410-04A_1x04_P2.54mm_Vertical, symbol Connector:Conn_01x04_Pin
- added R24, R26, R27, R30: 10k, Resistor_SMD:R_0805_2012Metric_Pad1.20x1.40mm_HandSolder, symbol Device:R
- added R28, R29, R31: 3.3M, Resistor_SMD:R_0805_2012Metric_Pad1.20x1.40mm_HandSolder, symbol Device:R
- added U6, U7: LM358DT, Package_SO:SOIC-8_3.9x4.9mm_P1.27mm, symbol LM358DT:LM358DT
- R13: value 10k -> 3.3M
Connections:
- net +5V: now also D2.1 (K), J19.1 (Pin_1), U6.8 (VCC+), U7.8 (VCC+); no longer C1.1, U3.4 (VCC), U3.6 (VCC)
- net GND: now also U1.9 (SDO/AD0), J19.2 (Pin_2), R28.1, R31.1, U6.4 (VCC-), U7.4 (VCC-)
- net UART RXD: now also J19.3 (Pin_3)
- net UART TXD: now also J19.4 (Pin_4)
- net V+: now also R26.1, R27.1
- net V1+: now also R30.1
- net V2+: now also R24.1; no longer R13.1
- net Vdiff: now also R29.1, U7.1 (OUT1)
- net Vdiff1: now also R13.1, U6.7 (OUT2)
- net Vdiff2: now also U6.1 (OUT1)
- net at R14.2, R15.2: now also U6.2 (IN1-)
- net at R16.2: now also R24.2, U6.3 (IN1+); no longer R13.2
- net at R10.2: now also R13.2, U6.5 (IN2+)
- new net: R30.2, R31.2, U6.6 (IN2-)
- new net: R27.2, R28.2, U7.2 (IN1-)
- new net: R26.2, R29.2, U7.3 (IN1+)
- new net: C1.1, D2.2 (A), U3.4 (VCC), U3.6 (VCC)
Other:
- moved on the sheet: C1, J10, J11, J13, R14, R15, R16, R19, R25, SW1

Commit message: Add files via upload
Parts:
- removed D2: MBR0520, Diode_SMD:D_SOD-123, symbol Diode:MBR0520
- added D3: MBR0520, Diode_SMD:D_SOD-123, symbol Diode:MBR0520
Connections:
- net +5V: now also C1.1, U3.4 (VCC), U3.6 (VCC), D3.1 (K); no longer J10.2 (VCC)
- new net: D3.2 (A), J10.2 (VCC)
Changed lines of the file:
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@@
 	)
 	(junction
-		(at 60.96 106.68)
-		(diameter 0)
-		(color 0 0 0 0)
-	)
-	(junction
 		(at 77.47 49.53)
 		(diameter 0)
@@
 	)
 	(junction
+		(at 60.96 106.68)
+		(diameter 0)
+		(color 0 0 0 0)
+	)
+	(junction
 		(at 237.49 137.16)
 		(diameter 0)
@@
 	(wire
 		(pts
-			(xy 251.46 91.44) (xy 251.46 95.25)
+			(xy 251.46 83.82) (xy 251.46 85.09)
 		)
 		(stroke
@@
 	(wire
 		(pts
+			(xy 251.46 92.71) (xy 251.46 95.25)
+		)
+		(stroke
+			(width 0)
+			(type default)
+		)
+	)
+	(wire
+		(pts
 			(xy 113.03 115.57) (xy 113.03 118.11)
 		)
@@
 	)
 	(label "ISP"
-		(at 254 83.82 0)
+		(at 261.62 83.82 0)
 		(effects
 			(font
@@
 	(symbol
 		(lib_id "power:+5V")
-		(at 251.46 91.44 0)
+		(at 251.46 83.82 0)
 		(unit 1)
 		(exclude_from_sim no)
@@
 		(fields_autoplaced yes)
 		(property "Reference" "#PWR0104"
-			(at 251.46 95.25 0)
+			(at 251.46 87.63 0)
 			(effects
 				(font
@@
 		)
 		(property "Value" "+5V"
-			(at 251.46 86.36 0)
+			(at 251.46 78.74 0)
 			(effects
 				(font
@@
 		)
 		(property "Footprint" ""
-			(at 251.46 91.44 0)
+			(at 251.46 83.82 0)
 			(effects
 				(font
@@
 		)
 		(property "Datasheet" ""
-			(at 251.46 91.44 0)
+			(at 251.46 83.82 0)
 			(effects
 				(font
@@
 		)
 		(property "Description" ""
-			(at 251.46 91.44 0)
+			(at 251.46 83.82 0)
 			(effects
 				(font
@@
 	(symbol
 		(lib_id "power:+5V")
-		(at 60.96 99.06 0)
+		(at 60.96 106.68 0)
 		(unit 1)
 		(exclude_from_sim no)
@@
 		(fields_autoplaced yes)
 		(property "Reference" "#PWR01"
-			(at 60.96 102.87 0)
+			(at 60.96 110.49 0)
 			(effects
 				(font
@@
 		)
 		(property "Value" "+5V"
-			(at 60.96 93.98 0)
+			(at 60.96 101.6 0)
 			(effects
 				(font
@@
 		)
 		(property "Footprint" ""
-			(at 60.96 99.06 0)
+			(at 60.96 106.68 0)
 			(effects
 				(font
@@
 		)
 		(property "Datasheet" ""
-			(at 60.96 99.06 0)
+			(at 60.96 106.68 0)
 			(effects
 				(font
@@
 		)
 		(property "Description" ""
-			(at 60.96 99.06 0)
+			(at 60.96 106.68 0)
 			(effects
 				(font
@@
 	)
 	(symbol
+		(lib_id "Diode:MBR0520")
+		(at 251.46 88.9 270)
+		(unit 1)
+		(exclude_from_sim no)
+		(in_bom yes)
+		(on_board yes)
+		(dnp no)
+		(property "Reference" "D3"
+			(at 253.492 84.582 90)
+			(effects
+				(font
+					(size 1.27 1.27)
+				)
+				(justify left)
+			)
+		)
+		(property "Value" "MBR0520"
+			(at 253.492 87.122 90)
+			(effects
+				(font
+					(size 1.27 1.27)
+				)
+				(justify left)
+			)
+		)
+		(property "Footprint" "Diode_SMD:D_SOD-123"
+			(at 247.015 88.9 0)
+			(effects
+				(font
+					(size 1.27 1.27)
+				)
+				(hide yes)
+			)
+		)
+		(property "Datasheet" "http://www.mccsemi.com/up_pdf/MBR0520~MBR0580(SOD123).pdf"
+			(at 251.46 88.9 0)
+			(effects
+				(font
+					(size 1.27 1.27)
+				)
+				(hide yes)
+			)
+		)
+		(property "Description" "20V 0.5A Schottky Power Rectifier Diode, SOD-123"
+			(at 251.46 88.9 0)
+			(effects
+				(font
+					(size 1.27 1.27)
+				)
+				(hide yes)
+			)
+		)
+		(pin "2"
+		)
+		(pin "1"
+		)
+		(instances
+			(project "445pcb_round3"
+				(path "/8efcc5b4-97b0-4b2b-85b0-3435af67eb97"
+					(reference "D3")
+					(unit 1)
+				)
+			)
+		)
+	)
+	(symbol
 		(lib_id "Device:R")
 		(at 167.64 101.6 90)
@@
 					(unit 1)
 				)
-			)
-		)
-	)
-	(symbol
-		(lib_id "Diode:MBR0520")
-		(at 60.96 102.87 270)
-		(unit 1)
-		(exclude_from_sim no)
-		(in_bom yes)
-		(on_board yes)
-		(dnp no)
-		(property "Reference" "D2"
-			(at 62.992 98.552 90)
-			(effects
-				(font
-					(size 1.27 1.27)
-				)
-				(justify left)
-			)
-		)
-		(property "Value" "MBR0520"
-			(at 62.992 101.092 90)
-			(effects
-				(font
-					(size 1.27 1.27)
-				)
-				(justify left)
-			)
-		)
-		(property "Footprint" "Diode_SMD:D_SOD-123"
-			(at 56.515 102.87 0)
-			(effects
-				(font
-					(size 1.27 1.27)
-				)
-				(hide yes)
-			)
-		)
-		(property "Datasheet" "http://www.mccsemi.com/up_pdf/MBR0520~MBR0580(SOD123).pdf"
-			(at 60.96 102.87 0)
-			(effects
-				(font
-					(size 1.27 1.27)
-				)
-				(hide yes)
-			)
-		)
-		(property "Description" "20V 0.5A Schottky Power Rectifier Diode, SOD-123"
-			(at 60.96 102.87 0)
-			(effects
-				(font
-					(size 1.27 1.27)
-				)
-				(hide yes)
-			)
-		)
-		(pin "2"
-		)
-		(pin "1"
-		)
-		(instances
-			(project ""
-				(path "/8efcc5b4-97b0-4b2b-85b0-3435af67eb97"
-					(reference "D2")
-					(unit 1)
-				)
